Commit message: pattern material included, for soft object

File: src/NUSENSE_description/urdf/materials.xacro (robot description, xacro)
@@ -10,3 +10,7 @@
   <color rgba="0.73725 0.69020 0.69020 0.71"/>
 </material>
+<material name="NUSENSE">
+  <texture filename="package://NUSENSE_description/urdf/textures/checkerboard_NUSENSE.png" />
+</material>
+<!-- to apply it onto future soft elasomer    -->
 </robot>
